File: inverter/inverter/inverter.sch (KiCad schematic (older format))
At the start: 6 parts, among them J1 in, J2 VDD, J3 VSS, J4 out, P1 P

Commit message: Created buffer and updated file organisation
Parts:
- removed N1: N, TO_SOT_Packages_SMD:TSOT-23, symbol Device:Q_NMOS_GSD
- removed P1: P, TO_SOT_Packages_SMD:TSOT-23, symbol Device:Q_PMOS_GSD
Connections:
- net labels added: VDD, VSS
- wire segments 12 -> 4
Changed lines of the file:
@@
 $Descr A4 11693 8268
 encoding utf-8
-Sheet 1 1
+Sheet 1 2
 Title ""
 Date ""
@@
 	1    0    0    -1
 $EndComp
+Wire Wire Line
+	4600 3150 4600 3050
+Wire Wire Line
+	4300 2300 3700 2300
+$Sheet
+S 4300 2100 550  400
+U 5AF22AE7
+F0 "Inv_1" 50
+F1 "lib/inverter.sch" 50
+F2 "in" I L 4300 2300 50
+F3 "out" O R 4850 2300 50
+$EndSheet
 $Comp
-L Device:Q_NMOS_GSD N1
-U 1 1 5AEFF8F6
-P 4500 2700
-F 0 "N1" H 4706 2746 50  0000 L CNN
-F 1 "N" H 4706 2655 50  0000 L CNN
-F 2 "TO_SOT_Packages_SMD:TSOT-23" H 4700 2800 50  0001 C CNN
-F 3 "~" H 4500 2700 50  0001 C CNN
-	1    4500 2700
-	1    0    0    -1
+L power:VDD #PWR0101
+U 1 1 5AF22C9D
+P 4600 1550
+F 0 "#PWR0101" H 4600 1400 50  0001 C CNN
+F 1 "VDD" H 4618 1723 50  0000 C CNN
+F 2 "" H 4600 1550 50  0001 C CNN
+F 3 "" H 4600 1550 50  0001 C CNN
+	1    4600 1550
+	-1   0    0    1
 $EndComp
+Wire Wire Line
+	4600 1550 4600 1450
 $Comp
-L Device:Q_PMOS_GSD P1
-U 1 1 5AEFFAFC
-P 4500 1900
-F 0 "P1" H 4706 1946 50  0000 L CNN
-F 1 "P" H 4706 1855 50  0000 L CNN
-F 2 "TO_SOT_Packages_SMD:TSOT-23" H 4700 2000 50  0001 C CNN
-F 3 "~" H 4500 1900 50  0001 C CNN
-	1    4500 1900
+L power:VSS #PWR0102
+U 1 1 5AF22D5E
+P 4600 3050
+F 0 "#PWR0102" H 4600 2900 50  0001 C CNN
+F 1 "VSS" H 4617 3223 50  0000 C CNN
+F 2 "" H 4600 3050 50  0001 C CNN
+F 3 "" H 4600 3050 50  0001 C CNN
+	1    4600 3050
 	1    0    0    -1
 $EndComp
 Wire Wire Line
-	4600 2100 4950 2100
-Wire Wire Line
-	4950 2100 4950 2300
-Wire Wire Line
-	4950 2300 5250 2300
-Wire Wire Line
-	4600 2500 4950 2500
-Wire Wire Line
-	4950 2500 4950 2300
-Connection ~ 4950 2300
-Wire Wire Line
-	4600 1700 4600 1450
-Wire Wire Line
-	4600 3150 4600 2900
-Wire Wire Line
-	4300 1900 4100 1900
-Wire Wire Line
-	4100 1900 4100 2300
-Wire Wire Line
-	4100 2300 3700 2300
-Wire Wire Line
-	4100 2300 4100 2700
-Wire Wire Line
-	4100 2700 4300 2700
-Connection ~ 4100 2300
+	4850 2300 5250 2300
 $EndSCHEMATC
